Commit message: fix #6

File: opp_racecar.xacro (robot description, xacro)
@@ -19,5 +19,5 @@
   <link name="base_link">
     <visual>
-      <origin xyz="-0.1 0 ${ground_offset+height/2}"/>
+      <origin xyz="${wheelbase/2} 0 ${ground_offset+height/2}"/>
       <geometry>
         <box size="${wheelbase} ${width} ${height}"/>
@@ -29,5 +29,5 @@
     <parent link="base_link"/>
     <child link="laser_model"/>
-    <origin xyz="0 0 ${ground_offset+height+(laser_height/2)}"/>
+    <origin xyz="${laser_distance_from_base_link} 0 ${ground_offset+height+(laser_height/2)}"/>
   </joint>
   <link name="laser_model">
@@ -42,5 +42,5 @@
     <parent link="base_link"/>
     <child link="back_left_wheel"/>
-    <origin xyz="${-wheelbase/2-0.1} ${(wheel_length+width)/2} ${wheel_radius}"/>
+    <origin xyz="0 ${(wheel_length+width)/2} ${wheel_radius}"/>
   </joint>
   <link name="back_left_wheel">
@@ -56,5 +56,5 @@
     <parent link="base_link"/>
     <child link="back_right_wheel"/>
-    <origin xyz="${-wheelbase/2-0.1} ${-(wheel_length+width)/2} ${wheel_radius}"/>
+    <origin xyz="0 ${-(wheel_length+width)/2} ${wheel_radius}"/>
   </joint>
   <link name="back_right_wheel">
@@ -70,5 +70,5 @@
     <parent link="base_link"/>
     <child link="front_left_hinge"/>
-    <origin xyz="${wheelbase/2-0.1} ${(wheel_length+width)/2} ${wheel_radius}"/>
+    <origin xyz="${wheelbase} ${(wheel_length+width)/2} ${wheel_radius}"/>
   </joint>
   <link name="front_left_hinge"/>
@@ -89,5 +89,5 @@
     <parent link="base_link"/>
     <child link="front_right_hinge"/>
-    <origin xyz="${wheelbase/2-0.1} ${-(wheel_length+width)/2} ${wheel_radius}"/>
+    <origin xyz="${wheelbase} ${-(wheel_length+width)/2} ${wheel_radius}"/>
   </joint>
   <link name="front_right_hinge"/>

Commit message: update xacro files

File: opp_racecar.xacro (robot description, xacro)
@@ -19,5 +19,5 @@
   <link name="base_link">
     <visual>
-      <origin xyz="-0.1 0 ${ground_offset+height/2}"/>
+      <origin xyz="{wheelbase/2} 0 ${ground_offset+height/2}"/>
       <geometry>
         <box size="${wheelbase} ${width} ${height}"/>
@@ -29,5 +29,5 @@
     <parent link="base_link"/>
     <child link="laser_model"/>
-    <origin xyz="0 0 ${ground_offset+height+(laser_height/2)}"/>
+    <origin xyz="{laser_distance_from_base_link} 0 ${ground_offset+height+(laser_height/2)}"/>
   </joint>
   <link name="laser_model">
@@ -42,5 +42,5 @@
     <parent link="base_link"/>
     <child link="back_left_wheel"/>
-    <origin xyz="${-wheelbase/2-0.1} ${(wheel_length+width)/2} ${wheel_radius}"/>
+    <origin xyz="$0 ${(wheel_length+width)/2} ${wheel_radius}"/>
   </joint>
   <link name="back_left_wheel">
@@ -56,5 +56,5 @@
     <parent link="base_link"/>
     <child link="back_right_wheel"/>
-    <origin xyz="${-wheelbase/2-0.1} ${-(wheel_length+width)/2} ${wheel_radius}"/>
+    <origin xyz="$0 ${-(wheel_length+width)/2} ${wheel_radius}"/>
   </joint>
   <link name="back_right_wheel">
@@ -70,5 +70,5 @@
     <parent link="base_link"/>
     <child link="front_left_hinge"/>
-    <origin xyz="${wheelbase/2-0.1} ${(wheel_length+width)/2} ${wheel_radius}"/>
+    <origin xyz="${wheelbase} ${(wheel_length+width)/2} ${wheel_radius}"/>
   </joint>
   <link name="front_left_hinge"/>
@@ -89,5 +89,5 @@
     <parent link="base_link"/>
     <child link="front_right_hinge"/>
-    <origin xyz="${wheelbase/2-0.1} ${-(wheel_length+width)/2} ${wheel_radius}"/>
+    <origin xyz="${wheelbase} ${-(wheel_length+width)/2} ${wheel_radius}"/>
   </joint>
   <link name="front_right_hinge"/>

Commit message: xacro bug fix

File: opp_racecar.xacro (robot description, xacro)
@@ -19,5 +19,5 @@
   <link name="base_link">
     <visual>
-      <origin xyz="{wheelbase/2} 0 ${ground_offset+height/2}"/>
+      <origin xyz="${wheelbase/2} 0 ${ground_offset+height/2}"/>
       <geometry>
         <box size="${wheelbase} ${width} ${height}"/>
@@ -29,5 +29,5 @@
     <parent link="base_link"/>
     <child link="laser_model"/>
-    <origin xyz="{laser_distance_from_base_link} 0 ${ground_offset+height+(laser_height/2)}"/>
+    <origin xyz="${laser_distance_from_base_link} 0 ${ground_offset+height+(laser_height/2)}"/>
   </joint>
   <link name="laser_model">
@@ -42,5 +42,5 @@
     <parent link="base_link"/>
     <child link="back_left_wheel"/>
-    <origin xyz="$0 ${(wheel_length+width)/2} ${wheel_radius}"/>
+    <origin xyz="0 ${(wheel_length+width)/2} ${wheel_radius}"/>
   </joint>
   <link name="back_left_wheel">
@@ -56,5 +56,5 @@
     <parent link="base_link"/>
     <child link="back_right_wheel"/>
-    <origin xyz="$0 ${-(wheel_length+width)/2} ${wheel_radius}"/>
+    <origin xyz="0 ${-(wheel_length+width)/2} ${wheel_radius}"/>
   </joint>
   <link name="back_right_wheel">
