Commit message: Spin the wheels at the car's actual rolling rate
The bridge integrates a per-car wheel angle from the sim's longitudinal
speed (no-slip v/r; the ST model carries no wheel-speed states) and
publishes it on the wheel TFs: front wheels get steer-about-z composed
with roll about the steered axle, rear wheels pure roll. Wheel radius
0.051 m measured from the wheel glb meshes, scaled per platform by the
same factors racecar_mesh.xacro applies.

Rear wheels move off their fixed joints onto the same hinge pattern the
fronts use (fixed base->hinge at the hub + continuous hinge->wheel about
y) so the bridge can animate them without fighting the static TF from
robot_state_publisher.

The wheel glbs are baked from one source model at its posed orientation
in the USD scene, so each carries a different camber+toe tilt off its
true axle - visible standing still and a wobble cone once spinning. Each
wheel visual gets an exact per-wheel rpy counter-rotation, measured from
the mesh vertices by the new scripts/measure_wheel_alignment.py (PCA;
the axle is the thin principal axis). Rerun it after re-exporting
meshes, or have usd_to_mesh.py bake wheels in a canonical axle-on-y
pose to zero these out.

Also wrap robot_description in ParameterValue(value_type=str): launch
yaml-parses bare Command parameter values, so any "colon + space" in
the xacro output aborted the whole launch with "Unable to parse the
value of parameter robot_description as yaml" while already-spawned
nodes lived on as orphans.

Co-Authored-By: Claude Fable 5 <noreply@anthropic.com>

File: urdf/racecar_mesh.xacro (robot description, xacro)
@@ -4,4 +4,9 @@
   Written by scripts/usd_to_mesh.py from meshes/roboracer.usd. Re-run that script
   after changing the USD; hand edits here are lost on the next regeneration.
+  NOTE - the wheel-spin structure below (back_*_hinge links + continuous wheel
+  joints, animated by the gym bridge) is a hand edit that must be folded into
+  usd_to_mesh.py before the next regeneration. Avoid "colon + space" anywhere
+  in this file; unless robot_description is wrapped in ParameterValue, launch
+  yaml-parses the URDF string and a colon turns it into a mapping.
   Same link and joint names as urdf/ego_racecar.xacro so TF, the gym bridge and
   anything downstream keep working - only the geometry changed, from primitive
@@ -31,4 +36,22 @@
   </xacro:if>
   <xacro:property name="mesh_dir" value="package://f1tenth_gym_ros/meshes"/>
+  <!-- ============================ WHEEL ALIGNMENT ============================
+       Per-wheel visual rpy corrections [deg]. All four wheels are baked from the
+       same source model but at their posed orientation in the USD scene, so each
+       glb carries a slightly different camber+toe tilt off its true axle. Any
+       residual angle between the mesh axle and link y wobbles once the bridge
+       spins the wheel TF, so the corrections must be exact per wheel - these are
+       measured from the mesh geometry by scripts/measure_wheel_alignment.py
+       (rerun it and paste new values after re-exporting the meshes). -->
+  <xacro:property name="align_fl_deg" value="${[-3.574, 0.068, 2.177]}"/>
+  <xacro:property name="align_fr_deg" value="${[1.899, -0.046, 2.803]}"/>
+  <xacro:property name="align_rl_deg" value="${[-2.543, -0.005, -0.246]}"/>
+  <xacro:property name="align_rr_deg" value="${[2.932, 0.007, -0.290]}"/>
+  <!-- =========================================================================== -->
+  <xacro:property name="d2r" value="${pi / 180}"/>
+  <xacro:property name="align_fl" value="${align_fl_deg[0]*d2r} ${align_fl_deg[1]*d2r} ${align_fl_deg[2]*d2r}"/>
+  <xacro:property name="align_fr" value="${align_fr_deg[0]*d2r} ${align_fr_deg[1]*d2r} ${align_fr_deg[2]*d2r}"/>
+  <xacro:property name="align_rl" value="${align_rl_deg[0]*d2r} ${align_rl_deg[1]*d2r} ${align_rl_deg[2]*d2r}"/>
+  <xacro:property name="align_rr" value="${align_rr_deg[0]*d2r} ${align_rr_deg[1]*d2r} ${align_rr_deg[2]*d2r}"/>
   <material name="${car_name}_accent">
     <color rgba="$(arg accent_color)"/>
@@ -66,11 +89,20 @@
     </visual>
   </link>
-  <joint name="base_to_back_left_wheel" type="fixed">
+  <!-- Rear wheels hang off fixed hinge frames like the fronts do, so the bridge
+       can publish their rolling rotation (about y, the axle) as a plain TF. -->
+  <joint name="base_to_back_left_hinge" type="fixed">
     <parent link="${car_name}/base_link"/>
+    <child link="${car_name}/back_left_hinge"/>
+    <origin xyz="${s * -0.000833 - lr} ${s * 0.130772} ${s * 0.051076}"/>
+  </joint>
+  <link name="${car_name}/back_left_hinge"/>
+  <joint name="back_left_hinge_to_wheel" type="continuous">
+    <parent link="${car_name}/back_left_hinge"/>
     <child link="${car_name}/back_left_wheel"/>
-    <origin xyz="${s * -0.000833 - lr} ${s * 0.130772} ${s * 0.051076}"/>
+    <axis xyz="0 1 0"/>
   </joint>
   <link name="${car_name}/back_left_wheel">
     <visual>
+      <origin rpy="${align_rl}"/>
       <geometry>
         <mesh filename="${mesh_dir}/roboracer_wheel_rear_left.glb" scale="${s} ${s} ${s}"/>
@@ -78,11 +110,18 @@
     </visual>
   </link>
-  <joint name="base_to_back_right_wheel" type="fixed">
+  <joint name="base_to_back_right_hinge" type="fixed">
     <parent link="${car_name}/base_link"/>
+    <child link="${car_name}/back_right_hinge"/>
+    <origin xyz="${s * 0.000833 - lr} ${s * -0.132075} ${s * 0.050856}"/>
+  </joint>
+  <link name="${car_name}/back_right_hinge"/>
+  <joint name="back_right_hinge_to_wheel" type="continuous">
+    <parent link="${car_name}/back_right_hinge"/>
     <child link="${car_name}/back_right_wheel"/>
-    <origin xyz="${s * 0.000833 - lr} ${s * -0.132075} ${s * 0.050856}"/>
+    <axis xyz="0 1 0"/>
   </joint>
   <link name="${car_name}/back_right_wheel">
     <visual>
+      <origin rpy="${align_rr}"/>
       <geometry>
         <mesh filename="${mesh_dir}/roboracer_wheel_rear_right.glb" scale="${s} ${s} ${s}"/>
@@ -105,4 +144,5 @@
   <link name="${car_name}/front_left_wheel">
     <visual>
+      <origin rpy="${align_fl}"/>
       <geometry>
         <mesh filename="${mesh_dir}/roboracer_wheel_front_left.glb" scale="${s} ${s} ${s}"/>
@@ -123,4 +163,5 @@
   <link name="${car_name}/front_right_wheel">
     <visual>
+      <origin rpy="${align_fr}"/>
       <geometry>
         <mesh filename="${mesh_dir}/roboracer_wheel_front_right.glb" scale="${s} ${s} ${s}"/>
